File: GarageMainBoard/GarageMainBoard.kicad_pcb (KiCad board)
At the start: 2 copper layers, 0 parts

Commit message: Main PCB start
Parts:
- added BZ1: Buzzer, Buzzers_Beepers:BUZZER, F.Cu at (110.4, 108.5)
- added C1: CP1, Capacitors_THT:CP_Radial_D10.0mm_P2.50mm, F.Cu at (87.5, 65.0)
- added C2: 100n, Capacitors_SMD:C_0805_HandSoldering, F.Cu at (108.0, 71.5)
- added C3: 10u, Capacitors_SMD:C_0805_HandSoldering, F.Cu at (100.5, 71.5)
- added C4: 100u, Capacitors_SMD:C_0805_HandSoldering, F.Cu at (91.5, 79.0)
- added C5: 100n, Capacitors_SMD:C_0805_HandSoldering, F.Cu at (79.0, 98.0)
- added J1: Conn_01x02, Pin_Headers:Pin_Header_Straight_1x02, F.Cu at (135.0, 75.5)
- added J2: Barrel_Jack, Connectors:BARREL_JACK, F.Cu at (69.8, 66.0)
- added J3: Conn_02x13_Odd_Even, Pin_Headers:Pin_Header_Straight_2x13, F.Cu at (146.5, 87.3)
- added J4: Front_Panel_Connector, Connectors_JST:JST_PH_B8B-PH-K_08x2.00mm_Straight, F.Cu at (120.5, 89.0)
- added J5: RJ45, KevinLibrary:RJ45_LOW_PROFILE_NO_CUT, F.Cu at (64.5, 87.5)
- added J6: RJ45, KevinLibrary:RJ45_LOW_PROFILE_NO_CUT, F.Cu at (64.5, 112.5)
- added Q1: IRLML6344, TO_SOT_Packages_SMD:SOT-23_Handsoldering, F.Cu at (94.5, 85.0)
- added Q2: IRLML6344, TO_SOT_Packages_SMD:SOT-23_Handsoldering, F.Cu at (94.5, 108.0)
- added Q3: IRLML6344, TO_SOT_Packages_SMD:SOT-23_Handsoldering, F.Cu at (88.0, 85.0)
- added R1: 100R, Resistors_SMD:R_0805_HandSoldering, F.Cu at (135.0, 87.5)
- added R10: 100R, Resistors_SMD:R_0805_HandSoldering, F.Cu at (94.2, 115.0)
- added R11: 100K, Resistors_SMD:R_0805_HandSoldering, F.Cu at (94.0, 120.0)
- added R12: 100R, Resistors_SMD:R_0805_HandSoldering, F.Cu at (88.0, 91.5)
- added R13: 1K, Resistors_SMD:R_0805_HandSoldering, F.Cu at (110.5, 120.0)
- added R14: 100K, Resistors_SMD:R_0805_HandSoldering, F.Cu at (88.0, 96.0)
- added R15: 1K, Resistors_SMD:R_0805_HandSoldering, F.Cu at (79.0, 94.0)
- added R2: 100R, Resistors_SMD:R_0805_HandSoldering, F.Cu at (135.0, 92.5)
- added R3: 100R, Resistors_SMD:R_0805_HandSoldering, F.Cu at (135.0, 97.0)
- added R4: 100R, Resistors_SMD:R_0805_HandSoldering, F.Cu at (135.0, 102.0)
- added R5: 100R, Resistors_SMD:R_0805_HandSoldering, F.Cu at (135.0, 106.0)
- added R6: 100R, Resistors_SMD:R_0805_HandSoldering, F.Cu at (135.0, 110.0)
- added R7: 1OOR, Resistors_SMD:R_0805_HandSoldering, F.Cu at (135.0, 114.5)
- added R8: 100R, Resistors_SMD:R_0805_HandSoldering, F.Cu at (94.5, 92.0)
- added R9: 100K, Resistors_SMD:R_0805_HandSoldering, F.Cu at (94.5, 96.0)
- added U1: AP1117-33, TO_SOT_Packages_SMD:SOT-223-3Lead_TabPin2, F.Cu at (104.5, 64.0)
- added U2: uClamp3306, KevinLibrary:SLP1616P6, F.Cu at (78.5, 87.7)
- added U3: uClamp3306, KevinLibrary:SLP1616P6, F.Cu at (78.0, 112.5)
