File: GarageMainBoard/GarageMainBoard.sch (KiCad schematic (older format))
At the start: 39 parts, among them J1 Conn_01x02, J2 Barrel_Jack, J3 Conn_02x13_Odd_Even, J4 Front_Panel_Connector, J5 RJ45, J6 RJ45, J7 5V Jumper, Q1 IRLML6344, Q2 IRLML6344, Q3 IRLML6344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

Commit message: Pull Ups on 365
Parts:
- added R16, R7: 1K, Resistors_SMD:R_0805_HandSoldering, symbol R
- J1, J7: footprint Pin_Headers:Pin_Header_Straight_1x02 -> Pin_Headers:Pin_Header_Straight_1x02_Pitch2.54mm
- J3: footprint Pin_Headers:Pin_Header_Straight_2x13 -> Pin_Headers:Pin_Header_Angled_2x13_Pitch2.54mm
- U1: footprint MODULE -> Housings_SOIC:SOIC-16_3.9x9.9mm_Pitch1.27mm
- U2: footprint (none) -> TO_SOT_Packages_SMD:SOT-353_SC-70-5_Handsoldering
- U5: footprint MODULE -> TO_SOT_Packages_SMD:SOT-353_SC-70-5_Handsoldering
Connections:
- wire segments 153 -> 155
Other:
- moved on the sheet: C2
Changed lines of the file:
@@
 F 0 "J3" H 2300 4550 50  0000 C CNN
 F 1 "Conn_02x13_Odd_Even" H 2300 3150 50  0000 C CNN
-F 2 "Pin_Headers:Pin_Header_Straight_2x13" H 2250 3850 50  0001 C CNN
+F 2 "Pin_Headers:Pin_Header_Angled_2x13_Pitch2.54mm" H 2250 3850 50  0001 C CNN
 F 3 "" H 2250 3850 50  0001 C CNN
 	1    2250 3850
@@
 F 0 "J1" H 1200 1500 50  0000 C CNN
 F 1 "Conn_01x02" H 1200 1200 50  0000 C CNN
-F 2 "Pin_Headers:Pin_Header_Straight_1x02" H 1200 1400 50  0001 C CNN
+F 2 "Pin_Headers:Pin_Header_Straight_1x02_Pitch2.54mm" H 1200 1400 50  0001 C CNN
 F 3 "" H 1200 1400 50  0001 C CNN
 	1    1200 1400
@@
 F 0 "J7" H 2800 3000 50  0000 C CNN
 F 1 "5V Jumper" H 2800 2700 50  0000 C CNN
-F 2 "Pin_Headers:Pin_Header_Straight_1x02" H 2800 2900 50  0001 C CNN
+F 2 "Pin_Headers:Pin_Header_Straight_1x02_Pitch2.54mm" H 2800 2900 50  0001 C CNN
 F 3 "" H 2800 2900 50  0001 C CNN
 	1    2800 2900
@@
 F 0 "U1" H 4100 1600 50  0000 C CNN
 F 1 "MC74HC365A" H 4100 1800 50  0000 C CNN
-F 2 "MODULE" H 4100 1700 50  0001 C CNN
+F 2 "Housings_SOIC:SOIC-16_3.9x9.9mm_Pitch1.27mm" H 4100 1700 50  0001 C CNN
 F 3 "DOCUMENTATION" H 4100 1700 50  0001 C CNN
 	1    4100 1700
@@
 L C C2
 U 1 1 5AC6FAB1
-P 5300 950
-F 0 "C2" H 5325 1050 50  0000 L CNN
-F 1 "100n" H 5325 850 50  0000 L CNN
-F 2 "Capacitors_SMD:C_0805_HandSoldering" H 5338 800 50  0001 C CNN
-F 3 "" H 5300 950 50  0001 C CNN
-	1    5300 950
-	0    1    1    0
+P 5500 1150
+F 0 "C2" H 5525 1250 50  0000 L CNN
+F 1 "100n" H 5525 1050 50  0000 L CNN
+F 2 "Capacitors_SMD:C_0805_HandSoldering" H 5538 1000 50  0001 C CNN
+F 3 "" H 5500 1150 50  0001 C CNN
+	1    5500 1150
+	-1   0    0    1
 $EndComp
 $Comp
@@
 $EndComp
 Wire Wire Line
-	5500 950  5500 1400
-Wire Wire Line
 	5000 1250 5000 1350
 Wire Wire Line
 	5000 1350 4850 1350
-Connection ~ 5000 1300
 Wire Wire Line
 	3350 2050 3200 2050
@@
 Wire Wire Line
 	4850 1450 5250 1450
-Wire Wire Line
-	5000 1300 5150 1300
-Wire Wire Line
-	5150 1300 5150 950
-Wire Wire Line
-	5500 950  5450 950
 Text Label 3050 1350 0    60   ~ 0
 ENABLE_1
@@
 F 0 "U2" H 7550 3275 60  0000 C CNN
 F 1 "CPDV5-3V3UP" H 8350 3300 60  0000 C CNN
-F 2 "" H 8000 3300 60  0001 C CNN
+F 2 "TO_SOT_Packages_SMD:SOT-353_SC-70-5_Handsoldering" H 8000 3300 60  0001 C CNN
 F 3 "" H 8000 3300 60  0001 C CNN
 	1    8000 3450
@@
 F 0 "U5" H 1750 6850 50  0000 C CNN
 F 1 "MC74VHC1GT50" H 1750 7050 50  0000 C CNN
-F 2 "MODULE" H 1750 6950 50  0001 C CNN
+F 2 "TO_SOT_Packages_SMD:SOT-353_SC-70-5_Handsoldering" H 1750 6950 50  0001 C CNN
 F 3 "DOCUMENTATION" H 1750 6950 50  0001 C CNN
 	1    1750 6950
@@
 Wire Wire Line
 	3450 6950 3450 7100
+$Comp
+L +3.3V #PWR038
+U 1 1 5AC84109
+P 5250 950
+F 0 "#PWR038" H 5250 800 50  0001 C CNN
+F 1 "+3.3V" H 5250 1090 50  0000 C CNN
+F 2 "" H 5250 950 50  0001 C CNN
+F 3 "" H 5250 950 50  0001 C CNN
+	1    5250 950
+	1    0    0    -1
+$EndComp
+$Comp
+L +3.3V #PWR039
+U 1 1 5AC84189
+P 5500 850
+F 0 "#PWR039" H 5500 700 50  0001 C CNN
+F 1 "+3.3V" H 5500 990 50  0000 C CNN
+F 2 "" H 5500 850 50  0001 C CNN
+F 3 "" H 5500 850 50  0001 C CNN
+	1    5500 850
+	1    0    0    -1
+$EndComp
+$Comp
+L +3.3V #PWR040
+U 1 1 5AC84209
+P 3000 900
+F 0 "#PWR040" H 3000 750 50  0001 C CNN
+F 1 "+3.3V" H 3000 1040 50  0000 C CNN
+F 2 "" H 3000 900 50  0001 C CNN
+F 3 "" H 3000 900 50  0001 C CNN
+	1    3000 900
+	1    0    0    -1
+$EndComp
+$Comp
+L R R16
+U 1 1 5AC84289
+P 5250 1200
+F 0 "R16" V 5330 1200 50  0000 C CNN
+F 1 "1K" V 5250 1200 50  0000 C CNN
+F 2 "Resistors_SMD:R_0805_HandSoldering" V 5180 1200 50  0001 C CNN
+F 3 "" H 5250 1200 50  0001 C CNN
+	1    5250 1200
+	-1   0    0    1
+$EndComp
+$Comp
+L R R7
+U 1 1 5AC843C9
+P 3000 1100
+F 0 "R7" V 3080 1100 50  0000 C CNN
+F 1 "1K" V 3000 1100 50  0000 C CNN
+F 2 "Resistors_SMD:R_0805_HandSoldering" V 2930 1100 50  0001 C CNN
+F 3 "" H 3000 1100 50  0001 C CNN
+	1    3000 1100
+	-1   0    0    1
+$EndComp
+Wire Wire Line
+	5500 1400 5500 1300
+Wire Wire Line
+	5500 1000 5500 850
+Wire Wire Line
+	5250 1050 5250 950
+Wire Wire Line
+	5250 1450 5250 1350
+Wire Wire Line
+	3000 950  3000 900
+Wire Wire Line
+	3000 1350 3000 1250
 $EndSCHEMATC

Commit message: PCB V2
Parts:
- J3: footprint Pin_Headers:Pin_Header_Angled_2x13_Pitch2.54mm -> Pin_Headers:Pin_Header_Straight_2x13_Pitch2.54mm
Changed lines of the file:
@@
 F 0 "J3" H 2300 4550 50  0000 C CNN
 F 1 "Conn_02x13_Odd_Even" H 2300 3150 50  0000 C CNN
-F 2 "Pin_Headers:Pin_Header_Angled_2x13_Pitch2.54mm" H 2250 3850 50  0001 C CNN
+F 2 "Pin_Headers:Pin_Header_Straight_2x13_Pitch2.54mm" H 2250 3850 50  0001 C CNN
 F 3 "" H 2250 3850 50  0001 C CNN
 	1    2250 3850
@@
 L +3.3V #PWR010
 U 1 1 5A5EE438
-P 7950 4800
-F 0 "#PWR010" H 7950 4650 50  0001 C CNN
-F 1 "+3.3V" H 7950 4940 50  0000 C CNN
-F 2 "" H 7950 4800 50  0001 C CNN
-F 3 "" H 7950 4800 50  0001 C CNN
-	1    7950 4800
+P 8200 4800
+F 0 "#PWR010" H 8200 4650 50  0001 C CNN
+F 1 "+3.3V" H 8200 4940 50  0000 C CNN
+F 2 "" H 8200 4800 50  0001 C CNN
+F 3 "" H 8200 4800 50  0001 C CNN
+	1    8200 4800
 	1    0    0    -1
 $EndComp
@@
 OPEN_HALL
 Wire Wire Line
-	8200 5200 8200 4700
-Wire Wire Line
 	8500 5200 8500 4700
-Text Label 8200 5200 1    60   ~ 0
+Text Label 7950 5200 1    60   ~ 0
 CLOSE_HALL
 Text Label 8500 5200 1    60   ~ 0
 OPEN_HALL
 Wire Wire Line
-	7950 4800 7950 5200
+	8200 4800 8200 5200
 $Comp
 L C C5
@@
 Wire Wire Line
 	2550 3650 3200 3650
-Text Label 3050 1650 0    60   ~ 0
+Text Label 3050 1450 0    60   ~ 0
 G_DOOR
 Text Label 2600 3650 0    60   ~ 0
@@
 Text Label 2650 3750 0    60   ~ 0
 LIGHT
-Text Label 3050 1450 0    60   ~ 0
+Text Label 3050 1650 0    60   ~ 0
 LIGHT
 $Comp
@@
 Wire Wire Line
 	4850 2050 5400 2050
-Text Label 3050 1550 0    60   ~ 0
+Text Label 3050 1750 0    60   ~ 0
 LIGHT_X
 Text Label 3050 2950 0    60   ~ 0
 LIGHT_X
-Text Label 3000 1750 0    60   ~ 0
+Text Label 3000 1550 0    60   ~ 0
 G_DOOR_X
 Text Label 4800 2950 0    60   ~ 0
 G_DOOR_X
-Text Label 3000 1950 0    60   ~ 0
+Text Label 3050 1950 0    60   ~ 0
 PIEZO_X
 Text Label 4350 5500 0    60   ~ 0
@@
 Wire Wire Line
 	3000 1350 3000 1250
+Wire Wire Line
+	7950 5200 7950 4700
 $EndSCHEMATC
